File: ifaces.kicad_sch (KiCad schematic)
At the start: 63 parts, among them J5 Vibrator, J6 Buzzer, J7 Display, J8 USB C, Q4 BSS138, Q5 BSS138, Q6 IRLML6401, Q7 BSS138, SW2 "OK", U6 USBLC6-2SC6

Commit message: fixes
- USB-C closer to the board's edge
- added 20pF caps for the 32.768kHz resonator
- replaced ferrite beads with 0805-sized ones
Parts:
- FB3: MPN 81-NFZ2MSD102SZ10L -> 810-MPZ2012S102AT000; PN 81-NFZ2MSD102SZ10L -> 810-MPZ2012S102AT000
Changed lines of the file:
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@@
 	(title_block
 		(title "Mainboard replacement for Nokia 3310")
-		(date "13-12-2024")
+		(date "24-01-2025")
 		(rev "Rev A")
 		(company "M17 Project")
@@
 	(label "ROW_3"
 		(at 254 118.11 0)
-		(fields_autoplaced yes)
 		(effects
 			(font
@@
 	(label "ROW_2"
 		(at 254 107.95 0)
-		(fields_autoplaced yes)
 		(effects
 			(font
@@
 	(label "{KEY_COLS}"
 		(at 259.08 151.13 180)
-		(fields_autoplaced yes)
 		(effects
 			(font
@@
 	(label "ROW_4"
 		(at 254 128.27 0)
-		(fields_autoplaced yes)
 		(effects
 			(font
@@
 	(label "COL_3"
 		(at 237.49 148.59 0)
-		(fields_autoplaced yes)
 		(effects
 			(font
@@
 	(label "ROW_5"
 		(at 254 138.43 0)
-		(fields_autoplaced yes)
 		(effects
 			(font
@@
 	(label "{KEY_ROWS}"
 		(at 251.46 90.17 180)
-		(fields_autoplaced yes)
 		(effects
 			(font
@@
 	(label "COL_2"
 		(at 224.79 148.59 0)
-		(fields_autoplaced yes)
 		(effects
 			(font
@@
 	(label "COL_1"
 		(at 212.09 148.59 0)
-		(fields_autoplaced yes)
 		(effects
 			(font
@@
 	(label "ROW_1"
 		(at 254 97.79 0)
-		(fields_autoplaced yes)
 		(effects
 			(font
@@
 		(shape bidirectional)
 		(at 223.52 43.18 180)
-		(fields_autoplaced yes)
 		(effects
 			(font
@@
 		(shape input)
 		(at 142.24 86.36 270)
-		(fields_autoplaced yes)
 		(effects
 			(font
@@
 		(shape input)
 		(at 67.31 101.6 180)
-		(fields_autoplaced yes)
 		(effects
 			(font
@@
 		(shape bidirectional)
 		(at 223.52 45.72 180)
-		(fields_autoplaced yes)
 		(effects
 			(font
@@
 		(shape output)
 		(at 234.95 90.17 180)
-		(fields_autoplaced yes)
 		(effects
 			(font
@@
 		(shape output)
 		(at 187.96 133.35 180)
-		(fields_autoplaced yes)
 		(effects
 			(font
@@
 		(shape input)
 		(at 147.32 86.36 270)
-		(fields_autoplaced yes)
 		(effects
 			(font
@@
 		(shape input)
 		(at 260.35 151.13 0)
-		(fields_autoplaced yes)
 		(effects
 			(font
@@
 		(shape input)
 		(at 132.08 86.36 270)
-		(fields_autoplaced yes)
 		(effects
 			(font
@@
 		(shape output)
 		(at 189.23 24.13 180)
-		(fields_autoplaced yes)
 		(effects
 			(font
@@
 		(shape input)
 		(at 144.78 86.36 270)
-		(fields_autoplaced yes)
 		(effects
 			(font
@@
 		(shape input)
 		(at 31.75 171.45 180)
-		(fields_autoplaced yes)
 		(effects
 			(font
@@
 		(shape input)
 		(at 139.7 86.36 270)
-		(fields_autoplaced yes)
 		(effects
 			(font
@@
 		(shape input)
 		(at 33.02 101.6 180)
-		(fields_autoplaced yes)
 		(effects
 			(font
@@
 			)
 		)
-		(property "PN" "81-NFZ2MSD102SZ10L"
+		(property "PN" "810-MPZ2012S102AT000"
 			(at 203.2 24.13 0)
 			(effects
@@
 			)
 		)
-		(property "MPN" "81-NFZ2MSD102SZ10L"
+		(property "MPN" "810-MPZ2012S102AT000"
 			(at 203.2 24.13 0)
 			(effects
